File: Rev2_F401RE/eagle/revb.brd (EAGLE design)
At the start: 96 x 73 mm, 162 parts, among them IC1 STM32F401RE, IC2 MCP73832, IC4 TPS63001, IC5 TPS63002, J1 USB4105-GF-A, J2 MEM2051-0019500A, J200 0, Q1 SI7615, T1 MMBTA06-7-F, T10 MMBTA06-7-F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

Commit message: Add barrel jack, add headers, add jumper between buck and rail, fix OLED pinout
Parts:
- added 3V3_EN, 5V_EN, 5V_OUT: (no value), pinhead:1X02
- added CN1: (no value), adafruit:DCJACK_2MM_PTH
Connections:
- new net 3V3_BUCK: 3V3_EN.2, C208.1, C209.1, C210.1, C211.1, IC4.1, IC4.10
- new net 5V_BUCK: 5V_EN.2, C215.1, C216.1, C217.1, C218.1, IC5.1, IC5.10
- new net GNDBREAK: CN1.GNDBREAK
- net +3V3: now also 3V3_EN.1; no longer C208.1, C209.1, C210.1, C211.1, IC4.1, IC4.10
- net +5V: now also 5V_EN.1, 5V_OUT.1; no longer C215.1, C216.1, C217.1, C218.1, IC5.1, IC5.10
- net GND: now also 5V_OUT.2, CN1.GND
- net USB_VIN: now also CN1.PWR
Routing:
- net 5V_BUCK: track 0.00 -> 6.22 mm, vias 0 -> 2
- net 3V3_BUCK: track 0.00 -> 6.06 mm, vias 0 -> 2
- net +5V: track 99.1 -> 103.1 mm, vias 20 -> 12
- net +3V3: track 64.0 -> 62.0 mm, vias 31 -> 23
- net SPKR_EN_BTN: track 45.1 -> 46.9 mm
- net TIM1_CH1: track 68.1 -> 67.3 mm
- added copper zone on layer 1, net 3V3_BUCK
- added copper zone on layer 1, net 5V_BUCK
- removed copper zone on layer 1, net +3V3
- removed copper zone on layer 1, net +5V

Commit message: Add IO for a relay board
Parts:
- removed 5V_OUT: (no value), pinhead:1X02
- added Q2: 2N3906, transistor-pnp:TO92
- added Q3: 2N3904, transistor-neu-to92:TO92
- added R151: 2k2, rcl:R0603
- added RELAY_CTL: (no value), adafruit:1X03
- moved OH_SHIT 5.30 mm to (83.8, 24.8), turned to 180 degrees
- moved R114 4.80 mm to (92.6, 21.9)
- moved R109 1.87 mm to (78.0, 25.2)
- renumbered R202\ to R202, R204\ to R204
Connections:
- new net RELAY: IC1.36, R151.2
- new net RELAY_OUT: Q2.1, Q3.1, RELAY_CTL.2
- new net RLY_BASE: Q2.2, Q3.2, R151.1
- net +3V3: now also Q2.3
- net +5V: no longer 5V_OUT.1
- net GND: now also Q3.3, RELAY_CTL.1; no longer 5V_OUT.2
- net USB_VIN: now also RELAY_CTL.3
Routing:
- net RELAY: track 0.00 -> 55.5 mm, vias 0 -> 2
- net RELAY_OUT: track 0.00 -> 14.3 mm
- net RLY_BASE: track 0.00 -> 10.7 mm
- net OH_SHIT_BTN: track 61.4 -> 70.2 mm
- net SDIO_D1: track 58.5 -> 59.8 mm
- net SDIO_DETECT: track 44.7 -> 43.9 mm
- net +3V3: track 62.0 -> 61.5 mm
- net GND: vias 321 -> 319
